File: Diseño CanSat UTN/Placa principal/Diseño CanSat UTN.kicad_pcb (KiCad board)
At the start: 2 copper layers, 60 x 60 mm, 10 parts, among them J1 Jack-DC, J2 Conn_01x15_MountingPin, J3 Conn_01x15_MountingPin, U1 L7805

Commit message: Subiendo Diseños
Parts:
- A1: footprint Module:Arduino_Nano -> Arduino Nano 3D:Arduino_Nano
- J1: footprint Connector_BarrelJack:BarrelJack_CUI_PJ-102AH_Horizontal -> Jack-DC:Jack-DC
- U1: footprint Package_TO_SOT_THT:TO-220-3_Vertical -> Package_TO_SOT_THT:TO-220-3_Horizontal_TabDown
- moved J1 45.7 mm to (169.5, 87.0)
- moved C4 28.2 mm to (154.4, 74.1), turned to 180 degrees
- moved C3 27.8 mm to (148.6, 74.1), turned to 180 degrees
- moved RV1 6.48 mm to (128.7, 114.1)
- moved U1 6.48 mm to (128.7, 104.1)
- moved C2 1.72 mm to (124.2, 96.6)
- moved C1 1.25 mm to (124.2, 103.6)
Connections:
- J1 pad 3: (no net) -> unconnected-(J1-Pad3)
Routing:
- net +9V: track 11.6 -> 84.8 mm
- net +5V: track 65.5 -> 81.3 mm
- net Net-(U1-IN): track 10.9 -> 9.71 mm

Commit message: Actualizando diseño
Parts:
- removed RV1: R_Potentiometer, Button_Switch_THT:SW_Push_2P2T_Toggle_CK_PVA2OAH5xxxxxxV2
- added S1: Switch-Horizontal, Switch-Horizontal:Switch-Horizontal, B.Cu at (177.0, 100.5)
- added U2: MicroSD-Card-Adapter, MicroSD-Card-Adapter:MicroSD-Card-Adapter, B.Cu at (135.0, 100.0)
Routing:
- net Net-(U1-IN): track 9.71 -> 87.5 mm
- net +9V: track 84.8 -> 30.1 mm

Commit message: actualizando diseños
Parts:
- S1: footprint Switch-Horizontal:Switch-Horizontal -> Switch-Horizontal:Switch-Horizontal-2
- moved S1 6.88 mm to (171.1, 104.1), turned to 90 degrees
- moved J1 5.58 mm to (168.0, 81.7)
Routing:
- net /Arduino Nano/14: track 3.67 -> 32.0 mm, vias 0 -> 1
- net /Arduino Nano/15: track 3.67 -> 31.7 mm
- net /Arduino Nano/7: track 3.67 -> 29.9 mm, vias 0 -> 2
- net +5V: track 81.3 -> 106.8 mm
- net /Arduino Nano/16: track 3.66 -> 28.0 mm
- net GND: track 7.33 -> 12.2 mm, vias 0 -> 1
- net +9V: track 30.1 -> 27.8 mm
- net Net-(U1-IN): track 87.5 -> 86.8 mm
- added copper zone on F.Cu, net GND

Commit message: ACTUALIZACION
Parts:
- removed J3: Conn_01x15_MountingPin, Connector_PinHeader_2.54mm:PinHeader_1x15_P2.54mm_Vertical
- removed S1: Switch-Horizontal, Switch-Horizontal:Switch-Horizontal-2
- removed U2: MicroSD-Card-Adapter, MicroSD-Card-Adapter:MicroSD-Card-Adapter
- added H1: MountingHole_Pad, MountingHole:MountingHole_2.2mm_M2_Pad, F.Cu at (156.0, 76.0)
- added H2: MountingHole_Pad, MountingHole:MountingHole_2.2mm_M2_Pad, F.Cu at (142.0, 76.0)
- added J5: Conn_01x15_MountingPin, Connector_PinHeader_2.54mm:PinHeader_1x15_P2.54mm_Vertical, F.Cu at (138.0, 83.5)
- added REF**: MountingHole_3.2mm_M3, MountingHole:MountingHole_3.2mm_M3, F.Cu at (131.0, 116.0)
- added REF**: MountingHole_3.2mm_M3, MountingHole:MountingHole_3.2mm_M3, F.Cu at (149.0, 76.0)
- added REF**: MountingHole_3.2mm_M3, MountingHole:MountingHole_3.2mm_M3, F.Cu at (167.0, 115.2)
- moved C4 42.2 mm to (130.0, 108.5), turned to -90 degrees
- moved C3 37.8 mm to (133.0, 108.5), turned to -90 degrees
- moved C1 23.9 mm to (132.0, 81.0), turned to -90 degrees
- moved C2 12.0 mm to (126.0, 108.5), turned to -90 degrees
- moved J1 4.47 mm to (167.0, 86.0)
- moved J2 2.72 mm to (160.0, 119.1)
- moved A1 2.59 mm to (141.4, 83.5)
- moved U1 1.73 mm to (127.5, 105.2)
Routing:
- net Net-(U1-IN): track 86.8 -> 39.6 mm
- net +5V: track 106.8 -> 62.6 mm
- net /Arduino Nano/14: track 32.0 -> 3.39 mm, vias 1 -> 0
- net /Arduino Nano/15: track 31.7 -> 3.39 mm
- net /Arduino Nano/7: track 29.9 -> 3.39 mm, vias 2 -> 0
- net /Arduino Nano/16: track 28.0 -> 3.37 mm
- net +9V: track 27.8 -> 16.9 mm
- net GND: track 12.2 -> 6.76 mm, vias 1 -> 0
- removed copper zone on F.Cu, net GND
Other:
- board size 60 x 60 mm -> 56 x 56 mm
