File: Diseño CanSat UTN/Placa principal/Fuente de alimentacion.kicad_sch (KiCad schematic)
At the start: 7 parts, among them J1 Jack-DC, U1 L7805

Commit message: Subiendo Diseños
Parts:
- J1: footprint Connector_BarrelJack:BarrelJack_CUI_PJ-102AH_Horizontal -> Jack-DC:Jack-DC; symbol Connector:Jack-DC -> Jack-DC:PJ-002A; Availability (none) -> In Stock; CUI_purchase_URL (none) -> https://www.cuidevices.com/product/interconnect/connectors/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; Check_prices (none) -> https://www.snapeda.com/parts/PJ-002A/CUI+Devices/view-part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; MANUFACTURER (none) -> CUI INC; MF (none) -> CUI Devices; MP (none) -> PJ-002A; Package (none) -> None; Price (none) -> None; Purchase-URL (none) -> https://pricing.snapeda.com/search?q=PJ-002A&ref=eda; STANDARD (none) -> Manufacturer recommendations; SnapEDA_Link (none) -> https://www.snapeda.com/parts/PJ-002A/CUI+Devices/view-part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
- U1: footprint Package_TO_SOT_THT:TO-220-3_Vertical -> Package_TO_SOT_THT:TO-220-3_Horizontal_TabDown
Connections:
- no-connect marks 1 -> 2
Changed lines of the file:
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@@
   (junction (at 124.206 59.182) (diameter 0) (color 0 0 0 0)
   )
+  (no_connect (at 66.802 61.722))
   (no_connect (at 83.566 62.992))
   (wire (pts (xy 133.096 69.088) (xy 133.096 68.072))
@@
     (stroke (width 0) (type default))
   )
-  (wire (pts (xy 69.596 59.182) (xy 69.342 59.182))
-    (stroke (width 0) (type default))
-  )
   (wire (pts (xy 109.474 66.802) (xy 109.474 69.088))
     (stroke (width 0) (type default))
@@
   )
   (wire (pts (xy 142.748 69.088) (xy 142.748 68.326))
-    (stroke (width 0) (type default))
-  )
-  (wire (pts (xy 69.596 64.262) (xy 69.342 64.262))
     (stroke (width 0) (type default))
   )
@@
     )
   )
-  (symbol (lib_id "power:GND") (at 69.596 64.262 0) (unit 1)
-    (in_bom yes) (on_board yes) (dnp no) (fields_autoplaced)
-    (property "Reference" "#PWR01" (at 69.596 70.612 0)
-      (effects (font (size 1.27 1.27)) hide)
-    )
-    (property "Value" "GND" (at 69.596 68.58 0)
-      (effects (font (size 1.27 1.27)))
-    )
-    (property "Footprint" "" (at 69.596 64.262 0)
-      (effects (font (size 1.27 1.27)) hide)
-    )
-    (property "Datasheet" "" (at 69.596 64.262 0)
+  (symbol (lib_id "power:GND") (at 66.802 64.262 0) (unit 1)
+    (in_bom yes) (on_board yes) (dnp no) (fields_autoplaced)
+    (property "Reference" "#PWR01" (at 66.802 70.612 0)
+      (effects (font (size 1.27 1.27)) hide)
+    )
+    (property "Value" "GND" (at 66.802 68.58 0)
+      (effects (font (size 1.27 1.27)))
+    )
+    (property "Footprint" "" (at 66.802 64.262 0)
+      (effects (font (size 1.27 1.27)) hide)
+    )
+    (property "Datasheet" "" (at 66.802 64.262 0)
       (effects (font (size 1.27 1.27)) hide)
     )
@@
     )
   )
-  (symbol (lib_id "Connector:Jack-DC") (at 61.722 61.722 0) (unit 1)
-    (in_bom yes) (on_board yes) (dnp no) (fields_autoplaced)
-    (property "Reference" "J1" (at 61.722 55.88 0)
+  (symbol (lib_id "Jack-DC:PJ-002A") (at 61.722 61.722 0) (unit 1)
+    (in_bom yes) (on_board yes) (dnp no) (fields_autoplaced)
+    (property "Reference" "J1" (at 58.4862 54.61 0)
       (effects (font (size 1.27 1.27)))
     )
@@
       (effects (font (size 1.27 1.27)) hide)
     )
-    (property "Footprint" "Connector_BarrelJack:BarrelJack_CUI_PJ-102AH_Horizontal" (at 62.992 62.738 0)
-      (effects (font (size 1.27 1.27)) hide)
-    )
-    (property "Datasheet" "~" (at 62.992 62.738 0)
-      (effects (font (size 1.27 1.27)) hide)
-    )
-    (pin "1")
-    (pin "2")
+    (property "Footprint" "Jack-DC:Jack-DC" (at 61.722 61.722 0)
+      (effects (font (size 1.27 1.27)) (justify bottom) hide)
+    )
+    (property "Datasheet" "~" (at 61.722 61.722 0)
+      (effects (font (size 1.27 1.27)) hide)
+    )
+    (property "MF" "CUI Devices" (at 61.722 61.722 0)
+      (effects (font (size 1.27 1.27)) (justify bottom) hide)
+    )
+    (property "Description" "2.0 x 6.5 mm, 2.5 A, Horizontal, Through Hole, Dc Power Jack Connector" (at 61.722 69.342 0)
+      (effects (font (size 1.27 1.27)) (justify bottom) hide)
+    )
+    (property "Package" "None" (at 61.722 61.722 0)
+      (effects (font (size 1.27 1.27)) (justify bottom) hide)
+    )
+    (property "Price" "None" (at 61.722 61.722 0)
+      (effects (font (size 1.27 1.27)) (justify bottom) hide)
+    )
+    (property "Check_prices" "https://www.snapeda.com/parts/PJ-002A/CUI+Devices/view-part/?ref=eda" (at 61.722 61.722 0)
+      (effects (font (size 1.27 1.27)) (justify bottom) hide)
+    )
+    (property "STANDARD" "Manufacturer recommendations" (at 61.722 61.722 0)
+      (effects (font (size 1.27 1.27)) (justify bottom) hide)
+    )
+    (property "SnapEDA_Link" "https://www.snapeda.com/parts/PJ-002A/CUI+Devices/view-part/?ref=snap" (at 61.722 61.722 0)
+      (effects (font (size 1.27 1.27)) (justify bottom) hide)
+    )
+    (property "MP" "PJ-002A" (at 61.722 61.722 0)
+      (effects (font (size 1.27 1.27)) (justify bottom) hide)
+    )
+    (property "Purchase-URL" "https://pricing.snapeda.com/search?q=PJ-002A&ref=eda" (at 61.722 61.722 0)
+      (effects (font (size 1.27 1.27)) (justify bottom) hide)
+    )
+    (property "CUI_purchase_URL" "https://www.cuidevices.com/product/interconnect/connectors/dc-power-connectors/jacks/pj-002a?utm_source=snapeda.com&utm_medium=referral&utm_campaign=snapedaBOM" (at 61.722 61.722 0)
+      (effects (font (size 1.27 1.27)) (justify bottom) hide)
+    )
+    (property "Availability" "In Stock" (at 61.722 61.722 0)
+      (effects (font (size 1.27 1.27)) (justify bottom) hide)
+    )
+    (property "MANUFACTURER" "CUI INC" (at 61.722 61.722 0)
+      (effects (font (size 1.27 1.27)) (justify bottom) hide)
+    )
+    (pin "1")
+    (pin "2")
+    (pin "3")
     (instances
       (project "Diseño CanSat UTN"
@@
       (effects (font (size 1.27 1.27)))
     )
-    (property "Footprint" "Package_TO_SOT_THT:TO-220-3_Vertical" (at 110.109 62.992 0)
+    (property "Footprint" "Package_TO_SOT_THT:TO-220-3_Horizontal_TabDown" (at 110.109 62.992 0)
       (effects (font (size 1.27 1.27) italic) (justify left) hide)
     )
@@
     )
   )
-  (symbol (lib_id "power:+9V") (at 69.596 59.182 0) (unit 1)
-    (in_bom yes) (on_board yes) (dnp no) (fields_autoplaced)
-    (property "Reference" "#PWR02" (at 69.596 62.992 0)
-      (effects (font (size 1.27 1.27)) hide)
-    )
-    (property "Value" "+9V" (at 69.596 54.61 0)
-      (effects (font (size 1.27 1.27)))
-    )
-    (property "Footprint" "" (at 69.596 59.182 0)
-      (effects (font (size 1.27 1.27)) hide)
-    )
-    (property "Datasheet" "" (at 69.596 59.182 0)
-      (effects (font (size 1.27 1.27)) hide)
-    )
+  (symbol (lib_id "power:+9V") (at 66.802 59.182 0) (unit 1)
+    (in_bom yes) (on_board yes) (dnp no) (fields_autoplaced)
+    (property "Reference" "#PWR02" (at 66.802 62.992 0)
+      (effects (font (size 1.27 1.27)) hide)
+    )
+    (property "Value" "+9V" (at 66.802 54.61 0)
+      (effects (font (size 1.27 1.27)))
+    )
+    (property "Footprint" "" (at 66.802 59.182 0)
+      (effects (font (size 1.27 1.27)) hide)
+    )
+    (property "Datasheet" "" (at 66.802 59.182 0)
+      (effects (font (size 1.27 1.27)) hide)
+    )

Commit message: Actualizando diseño
Parts:
- removed RV1: R_Potentiometer, Button_Switch_THT:SW_Push_2P2T_Toggle_CK_PVA2OAH5xxxxxxV2, symbol Device:R_Potentiometer
- added S1: Switch-Horizontal, Switch-Horizontal:Switch-Horizontal, symbol Switch-Horizontal:Switch-Horizontal
Connections:
- net +9V: now also S1.2
- net at C1.1, U1.1 (IN): now also S1.3
Changed lines of the file:
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@@
   )
   (no_connect (at 66.802 61.722))
-  (no_connect (at 83.566 62.992))
+  (no_connect (at 87.376 54.102))
   (wire (pts (xy 133.096 69.088) (xy 133.096 68.072))
     (stroke (width 0) (type default))
@@
     (stroke (width 0) (type default))
   )
+  (wire (pts (xy 72.136 53.848) (xy 72.136 56.642))
+    (stroke (width 0) (type default))
+  )
   (wire (pts (xy 94.742 59.182) (xy 94.742 59.944))
     (stroke (width 0) (type default))
@@
   (wire (pts (xy 87.376 59.182) (xy 94.742 59.182))
     (stroke (width 0) (type default))
-  )
-  (symbol (lib_id "power:+9V") (at 79.756 59.182 0) (unit 1)
-    (in_bom yes) (on_board yes) (dnp no) (fields_autoplaced)
-    (property "Reference" "#PWR03" (at 79.756 62.992 0)
-      (effects (font (size 1.27 1.27)) hide)
-    )
-    (property "Value" "+9V" (at 79.756 53.848 0)
-      (effects (font (size 1.27 1.27)))
-    )
-    (property "Footprint" "" (at 79.756 59.182 0)
-      (effects (font (size 1.27 1.27)) hide)
-    )
-    (property "Datasheet" "" (at 79.756 59.182 0)
-      (effects (font (size 1.27 1.27)) hide)
-    )
-    (pin "1")
-    (instances
-      (project "Diseño CanSat UTN"
-        (path "/6d01f5e8-1e9f-449b-95d5-6b60605ac758/43bc1217-1e03-40d2-83c7-fbb82912f4a3"
-          (reference "#PWR03") (unit 1)
-        )
-      )
-    )
   )
   (symbol (lib_id "power:GND") (at 94.742 69.088 0) (unit 1)
@@
     )
   )
-  (symbol (lib_id "Device:R_Potentiometer") (at 83.566 59.182 90) (mirror x) (unit 1)
-    (in_bom yes) (on_board yes) (dnp no) (fields_autoplaced)
-    (property "Reference" "RV1" (at 83.566 56.388 90)
-      (effects (font (size 1.27 1.27)))
-    )
-    (property "Value" "R_Potentiometer" (at 83.566 56.134 90)
-      (effects (font (size 1.27 1.27)) hide)
-    )
-    (property "Footprint" "Button_Switch_THT:SW_Push_2P2T_Toggle_CK_PVA2OAH5xxxxxxV2" (at 83.566 59.182 0)
-      (effects (font (size 1.27 1.27)) hide)
-    )
-    (property "Datasheet" "~" (at 83.566 59.182 0)
-      (effects (font (size 1.27 1.27)) hide)
+  (symbol (lib_id "Switch-Horizontal:Switch-Horizontal") (at 79.756 56.642 0) (unit 1)
+    (in_bom yes) (on_board yes) (dnp no)
+    (property "Reference" "S1" (at 79.756 48.26 0)
+      (effects (font (size 1.27 1.27)))
+    )
+    (property "Value" "Switch-Horizontal" (at 79.502 62.992 0)
+      (effects (font (size 1.27 1.27)))
+    )
+    (property "Footprint" "Switch-Horizontal:Switch-Horizontal" (at 79.756 56.642 0)
+      (effects (font (size 1.27 1.27)) (justify bottom) hide)
+    )
+    (property "Datasheet" "" (at 79.756 56.642 0)
+      (effects (font (size 1.27 1.27)) hide)
+    )
+    (property "MF" "E-Switch" (at 79.756 56.642 0)
+      (effects (font (size 1.27 1.27)) (justify bottom) hide)
+    )
+    (property "MAXIMUM_PACKAGE_HEIGHT" "6 mm" (at 79.756 56.642 0)
+      (effects (font (size 1.27 1.27)) (justify bottom) hide)
+    )
+    (property "Package" "None" (at 79.756 56.642 0)
+      (effects (font (size 1.27 1.27)) (justify bottom) hide)
+    )
+    (property "Price" "None" (at 79.756 56.642 0)
+      (effects (font (size 1.27 1.27)) (justify bottom) hide)
+    )
+    (property "Check_prices" "https://www.snapeda.com/parts/EG1206/E-Switch/view-part/?ref=eda" (at 79.756 56.642 0)
+      (effects (font (size 1.27 1.27)) (justify bottom) hide)
+    )
+    (property "STANDARD" "Manufacturer Recommendations" (at 79.756 56.642 0)
+      (effects (font (size 1.27 1.27)) (justify bottom) hide)
+    )
+    (property "PARTREV" "B" (at 79.756 56.642 0)
+      (effects (font (size 1.27 1.27)) (justify bottom) hide)
+    )
+    (property "SnapEDA_Link" "https://www.snapeda.com/parts/EG1206/E-Switch/view-part/?ref=snap" (at 79.756 56.642 0)
+      (effects (font (size 1.27 1.27)) (justify bottom) hide)
+    )
+    (property "MP" "EG1206" (at 79.756 56.642 0)
+      (effects (font (size 1.27 1.27)) (justify bottom) hide)
+    )
+    (property "Purchase-URL" "https://www.snapeda.com/api/url_track_click_mouser/?unipart_id=394778&manufacturer=E-Switch&part_name=EG1206&search_term=switch interruptor horizontal" (at 79.756 56.642 0)
+      (effects (font (size 1.27 1.27)) (justify bottom) hide)
+    )
+    (property "Description" "\nSWITCH SLIDE SPDT 200MA 30V\n" (at 79.756 56.642 0)
+      (effects (font (size 1.27 1.27)) (justify bottom) hide)
+    )
+    (property "MANUFACTURER" "E-Switch" (at 79.756 56.642 0)
+      (effects (font (size 1.27 1.27)) (justify bottom) hide)
+    )
+    (property "Availability" "In Stock" (at 79.756 56.642 0)
+      (effects (font (size 1.27 1.27)) (justify bottom) hide)
+    )
+    (property "SNAPEDA_PN" "EG1206" (at 79.756 56.642 0)
+      (effects (font (size 1.27 1.27)) (justify bottom) hide)
     )
     (pin "1")
@@
       (project "Diseño CanSat UTN"
         (path "/6d01f5e8-1e9f-449b-95d5-6b60605ac758/43bc1217-1e03-40d2-83c7-fbb82912f4a3"
-          (reference "RV1") (unit 1)
+          (reference "S1") (unit 1)
         )
       )
@@
         )
       )
+    )
+  )
+  (symbol (lib_id "power:+9V") (at 72.136 53.848 0) (unit 1)
+    (in_bom yes) (on_board yes) (dnp no) (fields_autoplaced)
+    (property "Reference" "#PWR03" (at 72.136 57.658 0)
+      (effects (font (size 1.27 1.27)) hide)
+    )
+    (property "Value" "+9V" (at 72.136 48.514 0)
+      (effects (font (size 1.27 1.27)))
+    )
+    (property "Footprint" "" (at 72.136 53.848 0)
+      (effects (font (size 1.27 1.27)) hide)
+    )
+    (property "Datasheet" "" (at 72.136 53.848 0)
+      (effects (font (size 1.27 1.27)) hide)
+    )
+    (pin "1")
+    (instances
+      (project "Diseño CanSat UTN"
+        (path "/6d01f5e8-1e9f-449b-95d5-6b60605ac758/43bc1217-1e03-40d2-83c7-fbb82912f4a3"
+          (reference "#PWR03") (unit 1)
+        )
+      )

Commit message: actualizando diseños
Parts:
- S1: footprint Switch-Horizontal:Switch-Horizontal -> Switch-Horizontal:Switch-Horizontal-2
Changed lines of the file:
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@@
       (effects (font (size 1.27 1.27)))
     )
-    (property "Footprint" "Switch-Horizontal:Switch-Horizontal" (at 79.756 56.642 0)
+    (property "Footprint" "Switch-Horizontal:Switch-Horizontal-2" (at 79.756 56.642 0)
       (effects (font (size 1.27 1.27)) (justify bottom) hide)
     )

Commit message: ACTUALIZACION
Parts:
- removed S1: Switch-Horizontal, Switch-Horizontal:Switch-Horizontal-2, symbol Switch-Horizontal:Switch-Horizontal
- added H1, H2: MountingHole_Pad, MountingHole:MountingHole_2.2mm_M2_Pad, symbol Mechanical:MountingHole_Pad
Connections:
- net +9V: now also H1.1
- net at C1.1, U1.1 (IN): now also H2.1
- no-connect marks 2 -> 1
Changed lines of the file:
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@@
   )
   (no_connect (at 66.802 61.722))
-  (no_connect (at 87.376 54.102))
   (wire (pts (xy 133.096 69.088) (xy 133.096 68.072))
     (stroke (width 0) (type default))
@@
     (stroke (width 0) (type default))
   )
-  (wire (pts (xy 87.376 59.182) (xy 94.742 59.182))
+  (wire (pts (xy 86.868 59.182) (xy 94.742 59.182))
     (stroke (width 0) (type default))
   )
@@
     )
   )
-  (symbol (lib_id "Switch-Horizontal:Switch-Horizontal") (at 79.756 56.642 0) (unit 1)
-    (in_bom yes) (on_board yes) (dnp no)
-    (property "Reference" "S1" (at 79.756 48.26 0)
-      (effects (font (size 1.27 1.27)))
-    )
-    (property "Value" "Switch-Horizontal" (at 79.502 62.992 0)
-      (effects (font (size 1.27 1.27)))
-    )
-    (property "Footprint" "Switch-Horizontal:Switch-Horizontal-2" (at 79.756 56.642 0)
-      (effects (font (size 1.27 1.27)) (justify bottom) hide)
-    )
-    (property "Datasheet" "" (at 79.756 56.642 0)
-      (effects (font (size 1.27 1.27)) hide)
-    )
-    (property "MF" "E-Switch" (at 79.756 56.642 0)
-      (effects (font (size 1.27 1.27)) (justify bottom) hide)
-    )
-    (property "MAXIMUM_PACKAGE_HEIGHT" "6 mm" (at 79.756 56.642 0)
-      (effects (font (size 1.27 1.27)) (justify bottom) hide)
-    )
-    (property "Package" "None" (at 79.756 56.642 0)
-      (effects (font (size 1.27 1.27)) (justify bottom) hide)
-    )
-    (property "Price" "None" (at 79.756 56.642 0)
-      (effects (font (size 1.27 1.27)) (justify bottom) hide)
-    )
-    (property "Check_prices" "https://www.snapeda.com/parts/EG1206/E-Switch/view-part/?ref=eda" (at 79.756 56.642 0)
-      (effects (font (size 1.27 1.27)) (justify bottom) hide)
-    )
-    (property "STANDARD" "Manufacturer Recommendations" (at 79.756 56.642 0)
-      (effects (font (size 1.27 1.27)) (justify bottom) hide)
-    )
-    (property "PARTREV" "B" (at 79.756 56.642 0)
-      (effects (font (size 1.27 1.27)) (justify bottom) hide)
-    )
-    (property "SnapEDA_Link" "https://www.snapeda.com/parts/EG1206/E-Switch/view-part/?ref=snap" (at 79.756 56.642 0)
-      (effects (font (size 1.27 1.27)) (justify bottom) hide)
-    )
-    (property "MP" "EG1206" (at 79.756 56.642 0)
-      (effects (font (size 1.27 1.27)) (justify bottom) hide)
-    )
-    (property "Purchase-URL" "https://www.snapeda.com/api/url_track_click_mouser/?unipart_id=394778&manufacturer=E-Switch&part_name=EG1206&search_term=switch interruptor horizontal" (at 79.756 56.642 0)
-      (effects (font (size 1.27 1.27)) (justify bottom) hide)
-    )
-    (property "Description" "\nSWITCH SLIDE SPDT 200MA 30V\n" (at 79.756 56.642 0)
-      (effects (font (size 1.27 1.27)) (justify bottom) hide)
-    )
-    (property "MANUFACTURER" "E-Switch" (at 79.756 56.642 0)
-      (effects (font (size 1.27 1.27)) (justify bottom) hide)
-    )
-    (property "Availability" "In Stock" (at 79.756 56.642 0)
-      (effects (font (size 1.27 1.27)) (justify bottom) hide)
-    )
-    (property "SNAPEDA_PN" "EG1206" (at 79.756 56.642 0)
-      (effects (font (size 1.27 1.27)) (justify bottom) hide)
+  (symbol (lib_id "power:GND") (at 66.802 64.262 0) (unit 1)
+    (in_bom yes) (on_board yes) (dnp no) (fields_autoplaced)
+    (property "Reference" "#PWR01" (at 66.802 70.612 0)
+      (effects (font (size 1.27 1.27)) hide)
+    )
+    (property "Value" "GND" (at 66.802 68.58 0)
+      (effects (font (size 1.27 1.27)))
+    )
+    (property "Footprint" "" (at 66.802 64.262 0)
+      (effects (font (size 1.27 1.27)) hide)
+    )
+    (property "Datasheet" "" (at 66.802 64.262 0)
+      (effects (font (size 1.27 1.27)) hide)
+    )
+    (pin "1")
+    (instances
+      (project "Diseño CanSat UTN"
+        (path "/6d01f5e8-1e9f-449b-95d5-6b60605ac758/43bc1217-1e03-40d2-83c7-fbb82912f4a3"
+          (reference "#PWR01") (unit 1)
+        )
+      )
+    )
+  )
+  (symbol (lib_id "Device:C") (at 142.748 64.516 0) (unit 1)
+    (in_bom yes) (on_board yes) (dnp no) (fields_autoplaced)
+    (property "Reference" "C4" (at 146.304 63.246 0)
+      (effects (font (size 1.27 1.27)) (justify left))
+    )
+    (property "Value" "C" (at 146.304 65.786 0)
+      (effects (font (size 1.27 1.27)) (justify left))
+    )
+    (property "Footprint" "Capacitor_THT:C_Rect_L4.6mm_W2.0mm_P2.50mm_MKS02_FKP02" (at 143.7132 68.326 0)
+      (effects (font (size 1.27 1.27)) hide)
+    )
+    (property "Datasheet" "~" (at 142.748 64.516 0)
+      (effects (font (size 1.27 1.27)) hide)
     )
     (pin "1")
     (pin "2")
-    (pin "3")
-    (instances
-      (project "Diseño CanSat UTN"
-        (path "/6d01f5e8-1e9f-449b-95d5-6b60605ac758/43bc1217-1e03-40d2-83c7-fbb82912f4a3"
-          (reference "S1") (unit 1)
-        )
-      )
-    )
-  )
-  (symbol (lib_id "power:GND") (at 66.802 64.262 0) (unit 1)
-    (in_bom yes) (on_board yes) (dnp no) (fields_autoplaced)
-    (property "Reference" "#PWR01" (at 66.802 70.612 0)
-      (effects (font (size 1.27 1.27)) hide)
-    )
-    (property "Value" "GND" (at 66.802 68.58 0)
-      (effects (font (size 1.27 1.27)))
-    )
-    (property "Footprint" "" (at 66.802 64.262 0)
-      (effects (font (size 1.27 1.27)) hide)
-    )
-    (property "Datasheet" "" (at 66.802 64.262 0)
-      (effects (font (size 1.27 1.27)) hide)
-    )
-    (pin "1")
-    (instances
-      (project "Diseño CanSat UTN"
-        (path "/6d01f5e8-1e9f-449b-95d5-6b60605ac758/43bc1217-1e03-40d2-83c7-fbb82912f4a3"
-          (reference "#PWR01") (unit 1)
-        )
-      )
-    )
-  )
-  (symbol (lib_id "Device:C") (at 142.748 64.516 0) (unit 1)
-    (in_bom yes) (on_board yes) (dnp no) (fields_autoplaced)
-    (property "Reference" "C4" (at 146.304 63.246 0)
-      (effects (font (size 1.27 1.27)) (justify left))
-    )
-    (property "Value" "C" (at 146.304 65.786 0)
-      (effects (font (size 1.27 1.27)) (justify left))
-    )
-    (property "Footprint" "Capacitor_THT:C_Rect_L4.6mm_W2.0mm_P2.50mm_MKS02_FKP02" (at 143.7132 68.326 0)
-      (effects (font (size 1.27 1.27)) hide)
-    )
-    (property "Datasheet" "~" (at 142.748 64.516 0)
-      (effects (font (size 1.27 1.27)) hide)
-    )
-    (pin "1")
-    (pin "2")
     (instances
       (project "Diseño CanSat UTN"
@@
         )
       )
+    )
+  )
+  (symbol (lib_id "Mechanical:MountingHole_Pad") (at 72.136 59.182 180) (unit 1)
+    (in_bom yes) (on_board yes) (dnp no) (fields_autoplaced)
+    (property "Reference" "H1" (at 74.93 59.182 0)
+      (effects (font (size 1.27 1.27)) (justify right))
+    )
+    (property "Value" "MountingHole_Pad" (at 74.93 61.722 0)
+      (effects (font (size 1.27 1.27)) (justify right))
+    )
+    (property "Footprint" "MountingHole:MountingHole_2.2mm_M2_Pad" (at 72.136 59.182 0)
+      (effects (font (size 1.27 1.27)) hide)
+    )
+    (property "Datasheet" "~" (at 72.136 59.182 0)
+      (effects (font (size 1.27 1.27)) hide)
+    )
+    (pin "1")
+    (instances
+      (project "Diseño CanSat UTN"
+        (path "/6d01f5e8-1e9f-449b-95d5-6b60605ac758/43bc1217-1e03-40d2-83c7-fbb82912f4a3"
+          (reference "H1") (unit 1)
+        )
+      )
+    )
+  )
+  (symbol (lib_id "Mechanical:MountingHole_Pad") (at 86.868 56.642 0) (unit 1)
+    (in_bom yes) (on_board yes) (dnp no) (fields_autoplaced)
+    (property "Reference" "H2" (at 89.662 54.102 0)
+      (effects (font (size 1.27 1.27)) (justify left))
+    )
+    (property "Value" "MountingHole_Pad" (at 89.662 56.642 0)
+      (effects (font (size 1.27 1.27)) (justify left))
+    )
+    (property "Footprint" "MountingHole:MountingHole_2.2mm_M2_Pad" (at 86.868 56.642 0)
+      (effects (font (size 1.27 1.27)) hide)
+    )
+    (property "Datasheet" "~" (at 86.868 56.642 0)
+      (effects (font (size 1.27 1.27)) hide)
+    )
+    (pin "1")
+    (instances
+      (project "Diseño CanSat UTN"
+        (path "/6d01f5e8-1e9f-449b-95d5-6b60605ac758/43bc1217-1e03-40d2-83c7-fbb82912f4a3"
+          (reference "H2") (unit 1)
+        )
+      )
