File: Diseño CanSat UTN/Placa de avisos/Placa de avisos.kicad_sch (KiCad schematic)
At the start: 15 parts, among them J1 Conn_01x15_MountingPin, J2 Conn_01x15_MountingPin

Commit message: ACTUALIZACION
Parts:
- removed D4, D5, D6: LED, LED_THT:LED_D5.0mm, symbol Device:LED
- removed R4, R5, R6: R, Resistor_THT:R_Axial_DIN0204_L3.6mm_D1.6mm_P5.08mm_Horizontal, symbol Device:R
Connections:
- net 14 is gone; now on net GND: J2.14 (Pin_14)
- net 19 is gone; now on net GND: J1.4 (Pin_4)
- net 10: now also R2.1; no longer BZ1.1 (-)
- net 11: no longer R1.1
- net 12: no longer R2.1
- net 13: no longer R3.1
- net 22: now also R1.1
- net 5: now also R3.1
- net 9: now also BZ1.1 (-)
- net GND: no longer J1.14 (Pin_14), J2.4 (Pin_4)
- new net 29: J1.14 (Pin_14)
- new net 4: J2.4 (Pin_4)
