File: Diseño CanSat UTN/Placa sensores/Placa de sensores/Placa de sensores.kicad_sch (KiCad schematic)
At the start: 4 parts, among them J2 Conn_01x15_MountingPin, J3 Conn_01x15_MountingPin, U1 BMP280

Commit message: ACTUALIZACION
Parts:
- added Q1: NPN, Package_TO_SOT_THT:TO-220-3_Horizontal_TabDown, symbol Simulation_SPICE:NPN
- added R1, R2: R, Resistor_THT:R_Axial_DIN0204_L3.6mm_D1.6mm_P7.62mm_Horizontal, symbol Device:R
Connections:
- net 14 is gone; now on net GND: J3.14 (Pin_14)
- net 19 is gone; now on net GND: J2.4 (Pin_4)
- net 12: now also R1.1
- net GND: now also R2.1; no longer J2.14 (Pin_14), J3.4 (Pin_4)
- new net: Q1.2 (B), R1.2
- new net: Q1.3 (E), R2.2
- new net +9V: Q1.1 (C)
- new net 29: J2.14 (Pin_14)
- new net 4: J3.4 (Pin_4)
Changed lines of the file:
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@@
   (no_connect (at 113.03 111.76))
   (no_connect (at 174.244 67.056))
-  (wire (pts (xy 166.878 100.076) (xy 169.164 100.076))
-    (stroke (width 0) (type default))
-  )
-  (wire (pts (xy 122.174 104.14) (xy 118.11 104.14))
+  (wire (pts (xy 194.818 66.04) (xy 194.818 65.024))
+    (stroke (width 0) (type default))
+  )
+  (wire (pts (xy 194.818 57.404) (xy 194.818 56.388))
+    (stroke (width 0) (type default))
+  )
+  (wire (pts (xy 175.514 51.308) (xy 178.054 51.308))
+    (stroke (width 0) (type default))
+  )
+  (wire (pts (xy 187.198 51.308) (xy 185.674 51.308))
+    (stroke (width 0) (type default))
+  )
+  (wire (pts (xy 123.444 78.74) (xy 118.11 78.74))
+    (stroke (width 0) (type default))
+  )
+  (wire (pts (xy 164.846 74.676) (xy 169.164 74.676))
+    (stroke (width 0) (type default))
+  )
+  (wire (pts (xy 194.818 44.704) (xy 194.818 46.228))
     (stroke (width 0) (type default))
   )
@@
   )
   (label "21" (at 118.11 83.82 0) (fields_autoplaced)
+    (effects (font (size 1.27 1.27)) (justify left bottom))
+  )
+  (label "12" (at 175.514 51.308 0) (fields_autoplaced)
     (effects (font (size 1.27 1.27)) (justify left bottom))
   )
@@
     )
   )
-  (symbol (lib_id "power:GND") (at 166.878 100.076 0) (unit 1)
-    (in_bom yes) (on_board yes) (dnp no) (fields_autoplaced)
-    (property "Reference" "#PWR02" (at 166.878 106.426 0)
-      (effects (font (size 1.27 1.27)) hide)
-    )
-    (property "Value" "GND" (at 166.878 105.41 0)
-      (effects (font (size 1.27 1.27)))
-    )
-    (property "Footprint" "" (at 166.878 100.076 0)
-      (effects (font (size 1.27 1.27)) hide)
-    )
-    (property "Datasheet" "" (at 166.878 100.076 0)
+  (symbol (lib_id "power:GND") (at 123.444 78.74 0) (unit 1)
+    (in_bom yes) (on_board yes) (dnp no) (fields_autoplaced)
+    (property "Reference" "#PWR03" (at 123.444 85.09 0)
+      (effects (font (size 1.27 1.27)) hide)
+    )
+    (property "Value" "GND" (at 123.444 83.82 0)
+      (effects (font (size 1.27 1.27)))
+    )
+    (property "Footprint" "" (at 123.444 78.74 0)
+      (effects (font (size 1.27 1.27)) hide)
+    )
+    (property "Datasheet" "" (at 123.444 78.74 0)
+      (effects (font (size 1.27 1.27)) hide)
+    )
+    (pin "1")
+    (instances
+      (project "Placa de sensores"
+        (path "/fa6e9766-9c9d-4c73-9cb8-9cce24517756"
+          (reference "#PWR03") (unit 1)
+        )
+      )
+    )
+  )
+  (symbol (lib_id "power:GND") (at 164.846 74.676 0) (unit 1)
+    (in_bom yes) (on_board yes) (dnp no) (fields_autoplaced)
+    (property "Reference" "#PWR02" (at 164.846 81.026 0)
+      (effects (font (size 1.27 1.27)) hide)
+    )
+    (property "Value" "GND" (at 164.846 79.756 0)
+      (effects (font (size 1.27 1.27)))
+    )
+    (property "Footprint" "" (at 164.846 74.676 0)
+      (effects (font (size 1.27 1.27)) hide)
+    )
+    (property "Datasheet" "" (at 164.846 74.676 0)
       (effects (font (size 1.27 1.27)) hide)
     )
@@
     )
   )
-  (symbol (lib_id "power:GND") (at 122.174 104.14 0) (unit 1)
-    (in_bom yes) (on_board yes) (dnp no) (fields_autoplaced)
-    (property "Reference" "#PWR03" (at 122.174 110.49 0)
-      (effects (font (size 1.27 1.27)) hide)
-    )
-    (property "Value" "GND" (at 122.174 109.22 0)
-      (effects (font (size 1.27 1.27)))
-    )
-    (property "Footprint" "" (at 122.174 104.14 0)
-      (effects (font (size 1.27 1.27)) hide)
-    )
-    (property "Datasheet" "" (at 122.174 104.14 0)
-      (effects (font (size 1.27 1.27)) hide)
-    )
-    (pin "1")
-    (instances
-      (project "Placa de sensores"
-        (path "/fa6e9766-9c9d-4c73-9cb8-9cce24517756"
-          (reference "#PWR03") (unit 1)
+  (symbol (lib_id "Device:R") (at 181.864 51.308 90) (unit 1)
+    (in_bom yes) (on_board yes) (dnp no) (fields_autoplaced)
+    (property "Reference" "R1" (at 181.864 45.72 90)
+      (effects (font (size 1.27 1.27)))
+    )
+    (property "Value" "R" (at 181.864 48.26 90)
+      (effects (font (size 1.27 1.27)))
+    )
+    (property "Footprint" "Resistor_THT:R_Axial_DIN0204_L3.6mm_D1.6mm_P7.62mm_Horizontal" (at 181.864 53.086 90)
+      (effects (font (size 1.27 1.27)) hide)
+    )
+    (property "Datasheet" "~" (at 181.864 51.308 0)
+      (effects (font (size 1.27 1.27)) hide)
+    )
+    (pin "1")
+    (pin "2")
+    (instances
+      (project "Placa de sensores"
+        (path "/fa6e9766-9c9d-4c73-9cb8-9cce24517756"
+          (reference "R1") (unit 1)
+        )
+      )
+    )
+  )
+  (symbol (lib_id "Device:R") (at 194.818 61.214 180) (unit 1)
+    (in_bom yes) (on_board yes) (dnp no) (fields_autoplaced)
+    (property "Reference" "R2" (at 197.0521 59.944 0)
+      (effects (font (size 1.27 1.27)) (justify right))
+    )
+    (property "Value" "R" (at 197.0521 62.484 0)
+      (effects (font (size 1.27 1.27)) (justify right))
+    )
+    (property "Footprint" "Resistor_THT:R_Axial_DIN0204_L3.6mm_D1.6mm_P7.62mm_Horizontal" (at 196.596 61.214 90)
+      (effects (font (size 1.27 1.27)) hide)
+    )
+    (property "Datasheet" "~" (at 194.818 61.214 0)
+      (effects (font (size 1.27 1.27)) hide)
+    )
+    (pin "1")
+    (pin "2")
+    (instances
+      (project "Placa de sensores"
+        (path "/fa6e9766-9c9d-4c73-9cb8-9cce24517756"
+          (reference "R2") (unit 1)
         )
       )
@@
     )
   )
+  (symbol (lib_id "Simulation_SPICE:NPN") (at 192.278 51.308 0) (unit 1)
+    (in_bom yes) (on_board yes) (dnp no) (fields_autoplaced)
+    (property "Reference" "Q1" (at 197.612 50.038 0)
+      (effects (font (size 1.27 1.27)) (justify left))
+    )
+    (property "Value" "NPN" (at 197.612 52.578 0)
+      (effects (font (size 1.27 1.27)) (justify left))
+    )
+    (property "Footprint" "Package_TO_SOT_THT:TO-220-3_Horizontal_TabDown" (at 255.778 51.308 0)
+      (effects (font (size 1.27 1.27)) hide)
+    )
+    (property "Datasheet" "~" (at 255.778 51.308 0)
+      (effects (font (size 1.27 1.27)) hide)
+    )
+    (property "Sim.Device" "NPN" (at 192.278 51.308 0)
+      (effects (font (size 1.27 1.27)) hide)
+    )
+    (property "Sim.Type" "GUMMELPOON" (at 192.278 51.308 0)
+      (effects (font (size 1.27 1.27)) hide)
+    )
+    (property "Sim.Pins" "1=C 2=B 3=E" (at 192.278 51.308 0)
+      (effects (font (size 1.27 1.27)) hide)
+    )
+    (pin "1")
+    (pin "2")
+    (pin "3")
+    (instances
+      (project "Placa de sensores"
+        (path "/fa6e9766-9c9d-4c73-9cb8-9cce24517756"
+          (reference "Q1") (unit 1)
+        )
+      )
+    )
+  )
   (symbol (lib_id "power:GND") (at 145.542 105.156 0) (unit 1)
     (in_bom yes) (on_board yes) (dnp no) (fields_autoplaced)
@@
     )
   )
+  (symbol (lib_id "power:+9V") (at 194.818 44.704 0) (unit 1)
+    (in_bom yes) (on_board yes) (dnp no) (fields_autoplaced)
+    (property "Reference" "#PWR06" (at 194.818 48.514 0)
+      (effects (font (size 1.27 1.27)) hide)
+    )
+    (property "Value" "+9V" (at 194.818 40.386 0)
+      (effects (font (size 1.27 1.27)))
+    )
+    (property "Footprint" "" (at 194.818 44.704 0)
+      (effects (font (size 1.27 1.27)) hide)
+    )
+    (property "Datasheet" "" (at 194.818 44.704 0)
+      (effects (font (size 1.27 1.27)) hide)
+    )
+    (pin "1")
+    (instances
+      (project "Placa de sensores"
+        (path "/fa6e9766-9c9d-4c73-9cb8-9cce24517756"
+          (reference "#PWR06") (unit 1)
+        )
+      )
+    )
+  )
   (symbol (lib_id "MPU5060:MPU6050") (at 145.542 94.996 0) (unit 1)
     (in_bom yes) (on_board yes) (dnp no) (fields_autoplaced)
@@
         )
       )
+    )
+  )
+  (symbol (lib_id "power:GND") (at 194.818 66.04 0) (unit 1)
+    (in_bom yes) (on_board yes) (dnp no) (fields_autoplaced)
+    (property "Reference" "#PWR05" (at 194.818 72.39 0)
+      (effects (font (size 1.27 1.27)) hide)
+    )
+    (property "Value" "GND" (at 194.818 70.866 0)
+      (effects (font (size 1.27 1.27)))
+    )
+    (property "Footprint" "" (at 194.818 66.04 0)
+      (effects (font (size 1.27 1.27)) hide)
+    )
+    (property "Datasheet" "" (at 194.818 66.04 0)
+      (effects (font (size 1.27 1.27)) hide)
+    )
+    (pin "1")
+    (instances
+      (project "Placa de sensores"
+        (path "/fa6e9766-9c9d-4c73-9cb8-9cce24517756"
+          (reference "#PWR05") (unit 1)
+        )
+      )
